Commit message: files updated with motors IDs

File: urdf/px.urdf (robot description, URDF)
Before this commit: robot px_robot, 7 links, 6 joints
Links:
- link base_link: geometry visual mesh filename=package://lab3_invkin_px_ros/meshes/Base.STL scale=1 1 1
- link link1: geometry visual mesh filename=package://lab3_invkin_px_ros/meshes/Shoulder.STL scale=1 1 1
- link link2: geometry visual mesh filename=package://lab3_invkin_px_ros/meshes/Bicep.STL scale=1 1 1
- link link3: geometry visual mesh filename=package://lab3_invkin_px_ros/meshes/Bicep.STL scale=1 1 1
- link link4: geometry visual mesh filename=package://lab3_invkin_px_ros/meshes/Wrist.STL scale=1 1 1

File: urdf/px_collision.urdf (robot description, URDF)
Before this commit: robot px_robot, 7 links, 6 joints
Links:
- link base_link: geometry collision mesh filename=package://lab3_invkin_px_ros/meshes/Base.STL scale=1 1 1; visual mesh filename=package://lab3_invkin_px_ros/meshes/Base.STL scale=1 1 1
- link link1: geometry collision mesh filename=package://lab3_invkin_px_ros/meshes/Shoulder.STL scale=1 1 1; visual mesh filename=package://lab3_invkin_px_ros/meshes/Shoulder.STL scale=1 1 1
- link link2: geometry collision mesh filename=package://lab3_invkin_px_ros/meshes/Bicep.STL scale=1 1 1; visual mesh filename=package://lab3_invkin_px_ros/meshes/Bicep.STL scale=1 1 1
- link link3: geometry collision mesh filename=package://lab3_invkin_px_ros/meshes/Bicep.STL scale=1 1 1; visual mesh filename=package://lab3_invkin_px_ros/meshes/Bicep.STL scale=1 1 1
- link link4: geometry collision mesh filename=package://lab3_invkin_px_ros/meshes/Wrist.STL scale=1 1 1; visual mesh filename=package://lab3_invkin_px_ros/meshes/Wrist.STL scale=1 1 1

File: urdf/px_transmission.urdf (robot description, URDF)
Before this commit: robot px_robot, 7 links, 6 joints
Links:
- link base_link: geometry visual mesh filename=package://lab3_invkin_px_ros/meshes/Base.STL scale=1 1 1
- link link1: geometry visual mesh filename=package://lab3_invkin_px_ros/meshes/Shoulder.STL scale=1 1 1
- link link2: geometry visual mesh filename=package://lab3_invkin_px_ros/meshes/Bicep.STL scale=1 1 1
- link link3: geometry visual mesh filename=package://lab3_invkin_px_ros/meshes/Bicep.STL scale=1 1 1
- link link4: geometry visual mesh filename=package://lab3_invkin_px_ros/meshes/Wrist.STL scale=1 1 1
